File: pcb/pcb.kicad_pcb (KiCad board)
At the start: 2 copper layers, 305 x 95.5 mm, 153 parts, among them J1 USB_C_Receptacle_USB2.0_14P, SW0 SW_Push, SW1 SW_Push_45deg, SW10 SW_Push_45deg, SW11 SW_Push_45deg, SW12 SW_Push_45deg, SW13 SW_Push_45deg, SW14 SW_Push_45deg, SW15 SW_Push_45deg, SW16 SW_Push_45deg, SW17 SW_Push_45deg, SW18 SW_Push_45deg, SW19 SW_Push_45deg, SW2 SW_Push_45deg, SW20 SW_Push_45deg, SW21 SW_Push_45deg, SW22 SW_Push_45deg, SW23 SW_Push_45deg, SW24 SW_Push_45deg, SW25 SW_Push_45deg, SW26 SW_Push_45deg, SW27 SW_Push_45deg, SW28 SW_Push_45deg, SW29 SW_Push_45deg, SW3 SW_Push_45deg, SW30 SW_Push_45deg, SW31 SW_Push_45deg, SW32 SW_Push_45deg, SW33 SW_Push_45deg, SW34 SW_Push_45deg, SW35 SW_Push_45deg, SW36 SW_Push_45deg, SW37 SW_Push_45deg, SW38 SW_Push_45deg, SW39 SW_Push_45deg, SW4 SW_Push_45deg, SW40 SW_Push_45deg, SW41 SW_Push_45deg, SW42 SW_Push_45deg, SW43 SW_Push_45deg, SW44 SW_Push_45deg, SW45 SW_Push_45deg, SW46 SW_Push_45deg, SW47 SW_Push_45deg, SW48 SW_Push_45deg, SW49 SW_Push_45deg, SW5 SW_Push_45deg, SW50 SW_Push_45deg, SW51 SW_Push_45deg, SW52 SW_Push_45deg, SW53 SW_Push_45deg, SW54 SW_Push_45deg, SW55 SW_Push_45deg, SW56 SW_Push_45deg, SW57 SW_Push_45deg, SW58 SW_Push_45deg, SW59 SW_Push_45deg, SW6 SW_Push_45deg, SW60 SW_Push_45deg, SW61 SW_Push_45deg, SW62 SW_Push_45deg, SW63 SW_Push_45deg, SW64 SW_Push_45deg, SW65 SW_Push_45deg, SW66 SW_Push_45deg, SW67 SW_Push_45deg, SW68 SW_Push_45deg, SW7 SW_Push_45deg, SW8 SW_Push_45deg, SW9 SW_Push_45deg, U1 ATmega32U4-A, Y1 16MHz

Commit message: Added Images - Finished Routing - Added silkscreen
Parts:
- added *: LOGO, LOGO, F.Cu at (33.9, 29.1)
- added *: LOGO, LOGO, B.Cu at (23.3, 32.0)
- added G***: LOGO, LOGO, F.Cu at (176.0, 96.0)
- added G***: LOGO, LOGO, B.Cu at (151.0, 96.0)
- C1, C2, C3, C4, C5, C6, R1, R2, R3, R4, R5, R6: moved to B.Cu
- J1: footprint Connector_USB:USB_C_Receptacle_HRO_TYPE-C-31-M-17 -> Connector_USB:USB_C_Receptacle_HRO_TYPE-C-31-M-12
- SW63, SW64, SW65: footprint Button_Switch_Keyboard:SW_Cherry_MX_1.00u_Plate -> Button_Switch_Keyboard:SW_Cherry_MX_1.00u_PCB
- moved D15 195.2 mm to (292.1, 18.3), turned to 90 degrees
- moved D30 194.8 mm to (297.7, 37.3), turned to 90 degrees
- moved R6 194.3 mm to (284.5, 14.1), turned to 90 degrees
- moved R1 187.7 mm to (282.5, 14.1), turned to -90 degrees
- moved R5 187.7 mm to (278.6, 14.1), turned to 90 degrees
- moved D58 187.1 mm to (301.6, 77.4), turned to 90 degrees
- moved R2 186.6 mm to (280.5, 14.2), turned to -90 degrees
- moved D68 186.3 mm to (301.6, 96.0), turned to 90 degrees
- moved D44 177.9 mm to (289.6, 57.1), turned to 90 degrees
- moved D29 170.1 mm to (273.1, 37.3), turned to 90 degrees
- moved D67 168.9 mm to (283.3, 96.0), turned to 90 degrees
- moved D57 168.4 mm to (282.6, 77.4), turned to 90 degrees
- moved D14 166.6 mm to (263.5, 18.3), turned to 90 degrees
- moved D66 151.2 mm to (264.3, 96.0), turned to 90 degrees
- moved D28 150.9 mm to (254.0, 37.3), turned to 90 degrees
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Routing:
- net GND: track 0.00 -> 573.5 mm, vias 0 -> 9
- net ROW1: track 0.00 -> 502.3 mm, vias 0 -> 1
- net ROW2: track 0.00 -> 387.8 mm, vias 0 -> 5
- net +5V: track 0.00 -> 353.7 mm, vias 0 -> 2
- net ROW3: track 0.00 -> 352.5 mm, vias 0 -> 5
- net Net-(U1-D+): track 0.00 -> 316.6 mm, vias 0 -> 8
- net ROW4: track 0.00 -> 307.5 mm, vias 0 -> 3
- net COLUMN8: track 0.00 -> 304.5 mm, vias 0 -> 8
- net COLUMN10: track 0.00 -> 297.8 mm, vias 0 -> 6
- net ROW5: track 0.00 -> 293.2 mm, vias 0 -> 1
- net COLUMN9: track 0.00 -> 288.9 mm, vias 0 -> 14
- net Net-(U1-D-): track 0.00 -> 278.6 mm, vias 0 -> 8
- net COLUMN14: track 0.00 -> 273.2 mm, vias 0 -> 2
- net COLUMN13: track 0.00 -> 262.4 mm, vias 0 -> 10
- net COLUMN12: track 0.00 -> 260.9 mm, vias 0 -> 9
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Other:
- board size 305 x 95.5 mm -> 305.6 x 103 mm
- board text added: "AMD X HACKCLUB"
- board text added: "Blueprint"
- board text added: "TAPS65"

Commit message: Rerouted - New Layout
Parts:
- added REF**: MountingHole_2.2mm_M2, MountingHole:MountingHole_2.2mm_M2, F.Cu at (0.62, 105.2)
- added REF**: MountingHole_2.2mm_M2, MountingHole:MountingHole_2.2mm_M2, F.Cu at (301.5, 105.2)
- added REF**: MountingHole_2.2mm_M2, MountingHole:MountingHole_2.2mm_M2, F.Cu at (0.62, 6.97)
- added REF**: MountingHole_2.2mm_M2, MountingHole:MountingHole_2.2mm_M2, F.Cu at (301.5, 6.97)
- SW14: footprint Button_Switch_Keyboard:SW_Cherry_MX_1.00u_PCB -> Button_Switch_Keyboard:SW_Cherry_MX_2.00u_PCB
- SW15: footprint Button_Switch_Keyboard:SW_Cherry_MX_2.00u_PCB -> Button_Switch_Keyboard:SW_Cherry_MX_1.00u_PCB
- SW29: footprint Button_Switch_Keyboard:SW_Cherry_MX_1.00u_PCB -> Button_Switch_Keyboard:SW_Cherry_MX_1.50u_PCB
- SW30: footprint Button_Switch_Keyboard:SW_Cherry_MX_1.50u_PCB -> Button_Switch_Keyboard:SW_Cherry_MX_1.00u_PCB
- SW43: footprint Button_Switch_Keyboard:SW_Cherry_MX_1.00u_PCB -> Button_Switch_Keyboard:SW_Cherry_MX_2.25u_PCB
- SW44: footprint Button_Switch_Keyboard:SW_Cherry_MX_2.25u_PCB -> Button_Switch_Keyboard:SW_Cherry_MX_1.00u_PCB
- moved D14 12.3 mm to (275.8, 18.3)
- moved SW14 12.3 mm to (270.4, 14.8)
- moved D44 11.9 mm to (301.5, 57.1)
- moved SW44 11.9 mm to (296.2, 52.9)
- moved SW43 11.8 mm to (265.4, 52.9)
- moved D43 11.8 mm to (271.3, 57.1)
- moved D15 9.56 mm to (301.7, 18.4)
- moved SW15 9.56 mm to (296.3, 14.9)
- moved F1 8.55 mm to (283.1, 15.9)
- moved R1 8.55 mm to (291.1, 14.2)
- moved R2 8.55 mm to (289.1, 14.4)
- moved R6 8.55 mm to (293.1, 14.2)
- moved R5 8.55 mm to (287.1, 14.2)
- moved J1 8.55 mm to (288.2, 7.25)
- moved SW30 4.77 mm to (296.2, 33.9)
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Routing:
- net GND: track 573.5 -> 347.7 mm, vias 9 -> 23
- net +5V: track 353.7 -> 286.3 mm, vias 2 -> 12
- net Net-(U1-D+): track 316.6 -> 272.9 mm, vias 8 -> 10
- net ROW3: track 352.5 -> 366.3 mm
- net ROW1: track 502.3 -> 512.5 mm, vias 1 -> 3
- net COLUMN15: track 244.9 -> 239.5 mm, vias 8 -> 12
- net Net-(J1-CC2): track 3.92 -> 9.20 mm, vias 2 -> 0
- net ROW2: track 387.8 -> 392.4 mm
- net Net-(U1-D-): track 278.6 -> 275.6 mm, vias 8 -> 7
- net COLUMN13: track 262.4 -> 264.4 mm
- net COLUMN14: track 273.2 -> 272.1 mm
- net Net-(F1-Pad1): track 12.1 -> 11.0 mm, vias 0 -> 3
- net Net-(D29-A): track 6.04 -> 6.68 mm
- net Net-(D14-A): track 6.19 -> 6.74 mm
Other:
- board size 305.6 x 103 mm -> 306.9 x 104.2 mm

Commit message: Updated Images
Parts:
- SW1, SW10, SW11, SW12, SW13, SW15, SW17, SW18, SW19, SW2, SW20, SW21, SW22, SW23, SW24, SW25, SW26, SW27, SW28, SW3, SW30, SW32, SW33, SW34, SW35, SW36, SW37, SW38, SW39, SW4, SW40, SW41, SW42, SW44, SW46, SW47, SW48, SW49, SW5, SW50, SW51, SW52, SW53, SW54, SW55, SW57, SW58, SW6, SW63, SW64, SW65, SW66, SW67, SW68, SW7, SW8, SW9: footprint Button_Switch_Keyboard:SW_Cherry_MX_1.00u_PCB -> Taps Keyboard shit:SW_Cherry_MX_1.00u_PCB
- SW14: footprint Button_Switch_Keyboard:SW_Cherry_MX_2.00u_PCB -> Taps Keyboard shit:SW_Cherry_MX_2.00u_PCB
- SW16, SW29: footprint Button_Switch_Keyboard:SW_Cherry_MX_1.50u_PCB -> Taps Keyboard shit:SW_Cherry_MX_1.50u_PCB
- SW31, SW56: footprint Button_Switch_Keyboard:SW_Cherry_MX_1.75u_PCB -> Taps Keyboard shit:SW_Cherry_MX_1.75u_PCB
- SW43, SW45: footprint Button_Switch_Keyboard:SW_Cherry_MX_2.25u_PCB -> Taps Keyboard shit:SW_Cherry_MX_2.25u_PCB
- SW59, SW60, SW61: footprint Button_Switch_Keyboard:SW_Cherry_MX_1.25u_PCB -> Taps Keyboard shit:SW_Cherry_MX_1.25u_PCB
- SW62: footprint Button_Switch_Keyboard:SW_Cherry_MX_6.25u_PCB -> Taps Keyboard shit:SW_Cherry_MX_6.25u_PCB
- moved SW56 6.21 mm to (248.3, 77.6)
- moved SW31 6.20 mm to (15.0, 58.6)
- moved SW16 5.68 mm to (12.7, 39.0)
- moved SW29 5.64 mm to (270.0, 38.8)
- moved SW14 2.73 mm to (267.7, 14.7)
- moved D14 2.73 mm to (273.1, 18.2)
- moved SW30 0.09 mm to (296.2, 33.8)
Routing:
- net +5V: track 286.3 -> 290.1 mm
- net COLUMN14: track 272.1 -> 273.8 mm, vias 2 -> 3
- net ROW1: track 512.5 -> 513.2 mm
