File: pcb/pcb.kicad_pcb (KiCad board)
At the start: 2 copper layers, 340.8 x 100 mm, 223 parts, among them SW1 SW_Push_45deg, SW10 SW_Push_45deg, SW11 SW_Push_45deg, SW12 SW_Push_45deg, SW13 SW_Push_45deg, SW14 SW_Push_45deg, SW15 SW_Push_45deg, SW16 SW_Push_45deg, SW17 SW_Push_45deg, SW18 SW_Push_45deg, SW19 SW_Push_45deg, SW2 SW_Push_45deg, SW20 SW_Push_45deg, SW21 SW_Push_45deg, SW22 SW_Push_45deg, SW23 SW_Push_45deg, SW24 SW_Push_45deg, SW25 SW_Push_45deg, SW26 SW_Push_45deg, SW27 SW_Push_45deg, SW28 SW_Push_45deg, SW29 SW_Push_45deg, SW3 SW_Push_45deg, SW30 SW_Push_45deg, SW31 SW_Push_45deg, SW32 SW_Push_45deg, SW33 SW_Push_45deg, SW34 SW_Push_45deg, SW35 SW_Push_45deg, SW36 SW_Push_45deg, SW37 SW_Push_45deg, SW38 SW_Push_45deg, SW39 SW_Push_45deg, SW4 SW_Push_45deg, SW40 SW_Push_45deg, SW41 SW_Push_45deg, SW42 SW_Push_45deg, SW43 SW_Push_45deg, SW44 SW_Push_45deg, SW45 SW_Push_45deg, SW46 SW_Push_45deg, SW47 SW_Push_45deg, SW48 SW_Push_45deg, SW49 SW_Push_45deg, SW5 SW_Push_45deg, SW50 SW_Push_45deg, SW51 SW_Push_45deg, SW52 SW_Push_45deg, SW53 SW_Push_45deg, SW54 SW_Push_45deg, SW55 SW_Push_45deg, SW56 SW_Push_45deg, SW57 SW_Push_45deg, SW58 SW_Push_45deg, SW59 SW_Push_45deg, SW6 SW_Push_45deg, SW60 SW_Push_45deg, SW61 SW_Push_45deg, SW62 SW_Push_45deg, SW63 SW_Push_45deg, SW64 SW_Push_45deg, SW65 SW_Push_45deg, SW66 SW_Push_45deg, SW67 SW_Push_45deg, SW68 SW_Push_45deg, SW7 SW_Push_45deg, SW8 SW_Push_45deg, SW9 SW_Push_45deg

Commit message: Fixed DRC issues
Parts:
- removed the G*** at (155.5, 100.4)
- added G***: LOGO, LOGO, B.Cu at (-5.56, 122.6)
- added G***: LOGO, LOGO, B.Cu at (-6.76, 141.5)
Routing:
- net ROW5: track 405.0 -> 417.1 mm
- net Net-(D112-DOUT): track 287.4 -> 297.6 mm
- net Net-(D130-DOUT): track 87.3 -> 97.1 mm
- net Net-(D82-DOUT): track 44.4 -> 51.8 mm
- net COLUMN15: track 475.9 -> 482.9 mm
- net Net-(D111-DOUT): track 49.3 -> 56.0 mm
- net Net-(D129-DOUT): track 91.7 -> 97.0 mm
- net ROW1: track 349.7 -> 354.6 mm
- net COLUMN12: track 367.1 -> 371.3 mm
- net Net-(D126-DOUT): track 296.7 -> 300.4 mm
- net ROW3: track 377.4 -> 381.0 mm
- net COLUMN13: track 413.0 -> 415.9 mm
- net ROW4: track 402.0 -> 404.8 mm
- net Net-(D110-DOUT): track 47.9 -> 50.3 mm
- net Net-(D81-DOUT): track 44.4 -> 46.5 mm
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